File: hardware/SignalForge_multipcb/SignalForge_multipcb.kicad_sch (KiCad schematic)
At the start: 62 parts, among them J1 Conn_01x08, J2 Micro_SD_Card_Det2, J3 Conn_02x15_Top_Bottom, P1 USB_C_Plug_USB2.0, Q1 AO3400A, Q2 SS8050, Q3 SS8050, SW1 BOOT, SW2 RST, SW3 SW_Push, SW4 SW_Push, SW5 SW_Push, SW6 SW_Push, U1 TP4057, U2 ESP32-S3-MINI-1, U3 USBLC6-2SC6, U4 TSDP343xx, U5 SPX3819M5-L-3-3, U6 CP2102N-Axx-xQFN28, U7 DM-OLED096-636

Commit message: add new design
Parts:
- added BOOT1, RESET1: ~, Button_Switch_SMD:SW_SPST_PTS810, symbol Switch:SW_MEC_5E
- added C1, C3, C4, C5: 0.1uF, Capacitor_SMD:C_0603_1608Metric, symbol Device:C_Small
- added C2, C6, C7: 10uF, Capacitor_SMD:C_0603_1608Metric, symbol Device:C_Small
- added D1: WS2812B, LED_SMD:LED_WS2812B_PLCC4_5.0x5.0mm_P3.2mm, symbol LED:WS2812B
- added D2: LED, LED_SMD:LED_0603_1608Metric, symbol Device:LED
- added J1, J3: ~, Connector_PinHeader_2.54mm:PinHeader_1x22_P2.54mm_Vertical, symbol Connector:Conn_01x22_Pin
- added JUSB1: USB_C_Receptacle_USB2.0, Connector_USB:USB_C_Receptacle_GCT_USB4105-xx-A_16P_TopMnt_Horizontal, symbol Connector:USB_C_Receptacle_USB2.0
- added R1, R2, R8: 5.1k, Resistor_SMD:R_0603_1608Metric, symbol Device:R_Small
- added R3, R4, R5: 10k, Resistor_SMD:R_0603_1608Metric, symbol Device:R_Small
- added R6: 1M, Resistor_SMD:R_0603_1608Metric, symbol Device:R_Small
- added R7: 200k, Resistor_SMD:R_0603_1608Metric, symbol Device:R_Small
- added U1: ESP32-S3-MINI-1-N8, ESP32-S3-MINI-1-N8:XCVR_ESP32-S3-MINI-1-N8, symbol ESP32-S3-MINI-1-N8:ESP32-S3-MINI-1-N8
- added U2: ESD7104MUTAG, Package_DFN_QFN:Diodes_UDFN-10_1.0x2.5mm_P0.5mm, symbol Power_Protection:D3V3XA4B10LP
- added U3: TLV75801PDRV, Package_SON:WSON-6-1EP_2x2mm_P0.65mm_EP1x1.6mm, symbol Regulator_Linear:TLV75801PDRV
- added U4: ENS210, Package_DFN_QFN:AMS_QFN-4-1EP_2x2mm_P0.95mm_EP0.7x1.6mm, symbol Sensor_Humidity:ENS210
- renumbered C13 to C10, C9 to C11, C14 to C12, C15 to C13, C11 to C14, C2 to C15, C3 to C2, C4 to C3, C5 to C4, C6 to C5, C7 to C6, C8 to C7, C10 to C8, C12 to C9, D6 to D1, D3 to D2, D4 to D3, D5 to D4, D1 to D5, D2 to D6, R17 to R1, R11 to R10, R13 to R11, R2 to R12, R3 to R13, R16 to R14, R14 to R15, R7 to R16, R15 to R17, R8 to R18, R9 to R19, R4 to R2, R5 to R3, R6 to R4, R12 to R5, R18 to R6, R19 to R7, R10 to R8, R1 to R9, SW3 to SW1, SW1 to SW2, SW4 to SW3, SW2 to SW4, U5 to U1, U1 to U2, U7 to U3, U2 to U5, U3 to U6, U6 to U7
Connections:
- net GND: now also BOOT1.1, BOOT1.2, C1.2, C2.2, C3.2, C4.2, C5.2, C6.2, C7.2, D1.3 (VSS), D2.1 (K), J1.22 (Pin_22), J3.1 (Pin_1), JUSB1.A1 (GND), JUSB1.A12 (GND), JUSB1.B1 (GND), JUSB1.B12 (GND), JUSB1.S1 (SHIELD), R1.2, R2.2, R7.1, RESET1.1, RESET1.2, U1.1 (GND), U1.2 (GND), U1.42 (GND), U1.43 (GND), U1.46 (GND), U1.47 (GND), U1.48 (GND), U1.49 (GND), U1.50 (GND), U1.51 (GND), U1.52 (GND), U1.53 (GND), U1.54 (GND), U1.55 (GND), U1.56 (GND), U1.57 (GND), U1.58 (GND), U1.59 (GND), U1.60 (GND), U1.61 (GND), U1.61_1 (GND), U1.61_2 (GND), U1.61_3 (GND), U1.61_4 (GND), U1.61_5 (GND), U1.61_6 (GND), U1.61_7 (GND), U1.61_8 (GND), U1.62 (GND), U1.63 (GND), U1.64 (GND), U1.65 (GND), U2.3 (VSS), U2.8 (VSS), U3.3 (GND), U3.7 (GND), U4.4 (GND), U4.5 (GND)
- new net: D2.2 (A), R8.2
- new net: JUSB1.B5 (CC2), R1.1
- new net: JUSB1.A5 (CC1), R2.1
- new net: R6.1, R7.2, U3.2 (FB)
- new net 3V3: C1.1, C2.1, C5.1, C7.1, D1.1 (VDD), J1.1 (Pin_1), R3.2, R4.2, R5.2, R6.2, R8.1, U1.3 (3V3), U3.1 (OUT), U4.1 (VDD)
- new net 5VUSB: C6.1, J1.21 (Pin_21), JUSB1.A4 (VBUS), JUSB1.A9 (VBUS), JUSB1.B4 (VBUS), JUSB1.B9 (VBUS), U2.4, U2.5, U2.7 (NC), U3.4 (EN), U3.6 (IN)
- new net ESP32_EN: C3.1, J3.2 (Pin_2), R3.1, RESET1.3 (K), RESET1.4 (A), U1.45 (EN)
- new net GPIO0: BOOT1.3 (K), BOOT1.4 (A), C4.1, J1.2 (Pin_2), U1.4 (IO0)
- new net GPIO1: J1.3 (Pin_3), U1.5 (IO1)
- new net GPIO10: J1.12 (Pin_12), U1.14 (IO10)
- new net GPIO11: J1.13 (Pin_13), U1.15 (IO11)
- new net GPIO12: J1.14 (Pin_14), U1.16 (IO12)
- new net GPIO13: J1.15 (Pin_15), U1.17 (IO13)
- new net GPIO14: J1.16 (Pin_16), U1.18 (IO14)
- new net GPIO15: J1.17 (Pin_17), U1.19 (IO15)
- new net GPIO16: J1.18 (Pin_18), U1.20 (IO16)
- new net GPIO2: J1.4 (Pin_4), U1.6 (IO2)
- new net GPIO21: J3.18 (Pin_18), U1.25 (IO21)
- new net GPIO26: J3.17 (Pin_17), U1.26 (IO26)
- new net GPIO3: J1.5 (Pin_5), U1.7 (IO3)
- new net GPIO33: J3.16 (Pin_16), U1.28 (IO33)
- new net GPIO34: J3.15 (Pin_15), U1.29 (IO34)
- new net GPIO35: J3.14 (Pin_14), U1.31 (IO35)
- new net GPIO36: J3.13 (Pin_13), U1.32 (IO36)
- new net GPIO37: J3.12 (Pin_12), U1.33 (IO37)
- new net GPIO38: J3.11 (Pin_11), U1.34 (IO38)
- new net GPIO39: J3.10 (Pin_10), U1.35 (IO39)
- new net GPIO4: J1.6 (Pin_6), U1.8 (IO4)
- new net GPIO40: J3.9 (Pin_9), U1.36 (IO40)
- new net GPIO41: J3.8 (Pin_8), U1.37 (IO41)
- new net GPIO42: J3.7 (Pin_7), U1.38 (IO42)
- new net GPIO45: J3.4 (Pin_4), U1.41 (IO45)
- new net GPIO46: J3.3 (Pin_3), U1.44 (IO46)
- new net GPIO47: J3.22 (Pin_22), U1.27 (IO47)
- new net GPIO48: D1.4 (DIN), J3.21 (Pin_21), U1.30 (IO48)
- new net GPIO5: J1.7 (Pin_7), U1.9 (IO5)
- new net GPIO6: J1.8 (Pin_8), U1.10 (IO6)
- new net GPIO7: J1.9 (Pin_9), U1.11 (IO7)
- new net GPIO8: J1.10 (Pin_10), U1.12 (IO8)
- new net GPIO9: J1.11 (Pin_11), U1.13 (IO9)
- new net I2C_SCL: J1.19 (Pin_19), R4.1, U1.21 (IO17), U4.2 (SCL)
- new net I2C_SDA: J1.20 (Pin_20), R5.1, U1.22 (IO18), U4.3 (SDA)
- new net RXD: J3.5 (Pin_5), U1.40 (RXD0)
- new net TXD: J3.6 (Pin_6), U1.39 (TXD0)
- new net USB_N: JUSB1.A7 (D-), JUSB1.B7 (D-), U1.23 (IO19), U2.2, U2.9 (NC)
- new net USB_P: JUSB1.A6 (D+), JUSB1.B6 (D+), U1.24 (IO20), U2.1, U2.10 (NC)
- no-connect marks 20 -> 25
Other:
- note added: "LED"
- moved on the sheet: BT1, C1, C10, C11, C12, C13, C14, C15, C2, C3, C4, C5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
